File: kicad/ebike-bsd.kicad_pcb (KiCad board)
At the start: 25 parts

Commit message: kicad: 生成器改两路设计, 重新生成工程文件
generate_kicad.py:
- MOSFET 符号 Q1-Q4 → Q1-Q2 (V2.6 同侧前后并联)
- 删除 R3/R4 栅极电阻及 R3/R4 junction
- 原理图标签 LED_FL/FR/RL/RR → LED_LEFT/RIGHT
- 原理图连线删除 Q3/Q4 栅极和 J6_3/4 输出
- PCB net 列表精简 (28 → 21), tracks 删除 Q3/Q4 走线
- J5 连接器 4pin → 3pin (L/R/GND), J6 4 端子 → 2 端子
- 内嵌 BOM 模板同步两路

重新生成 kicad/ 下工程文件 (BOM/sch/pcb), 与脚本一致
Parts:
- removed the ? at (0.00, 0.00) (x22)
- added ? (x4): , ['lib_id', ['str', 'Connector_Phoenix:TerminalBlock_Phoenix_MKDS_1x2_P5.08mm_Horizontal']], F.Cu at (0.00, 0.00)
- added ? (x4): , ['lib_id', ['str', 'R_Axial_DIN0207_L6.3mm_D2.5mm_P7.62mm_Horizontal']], F.Cu at (0.00, 0.00)
- added ? (x2): , ['lib_id', ['str', 'LED_D5.0mm']], F.Cu at (0.00, 0.00)
- added ? (x2): , ['lib_id', ['str', 'Connector_PinHeader_2.54mm:PinHeader_1x03_P2.54mm_Vertical']], F.Cu at (0.00, 0.00)
- added ? (x2): , ['lib_id', ['str', 'Connector_PinSocket_2.54mm:PinSocket_1x04_P2.54mm_Vertical']], F.Cu at (0.00, 0.00)
- added ? (x2): , ['lib_id', ['str', 'TO-220-3_Vertical']], F.Cu at (0.00, 0.00)
