File: kicad/ebike-bsd.kicad_pcb (KiCad board)
At the start: 25 parts

Commit message: Fix KiCad文件格式: 版本号20240108, 移除(str)包装, 兼容KiCad 8
Parts:
- removed ? (x6): , ['lib_id', ['str', 'Connector_Phoenix:TerminalBlock_Phoenix_MKDS_1x2_P5.08mm_Horizontal']]
- removed ? (x4): , ['lib_id', ['str', 'TO-220-3_Vertical']]
- removed ? (x6): , ['lib_id', ['str', 'R_Axial_DIN0207_L6.3mm_D2.5mm_P7.62mm_Horizontal']]
- removed ? (x2): , ['lib_id', ['str', 'LED_D5.0mm']]
- removed ?: , ['lib_id', ['str', 'Connector_PinHeader_2.54mm:PinHeader_1x05_P2.54mm_Vertical']]
- removed ?: , ['lib_id', ['str', 'Fuseholder_Cylinder-5x20mm']]
- removed ?: , ['lib_id', ['str', 'Connector_PinHeader_2.54mm:PinHeader_1x03_P2.54mm_Vertical']]
- removed ?: , ['lib_id', ['str', 'Connector_PinHeader_2.54mm:PinHeader_1x04_P2.54mm_Vertical']]
- removed ? (x2): , ['lib_id', ['str', 'Connector_PinSocket_2.54mm:PinSocket_1x04_P2.54mm_Vertical']]
- removed ?: , ['lib_id', ['str', 'Connector_PinSocket_2.54mm:PinSocket_2x19_P2.54mm_Vertical']]
- added D1, D2: , ['lib_id', 'LED_D5.0mm'], F.Cu at (0.00, 0.00)
- added F1: , ['lib_id', 'Fuseholder_Cylinder-5x20mm'], F.Cu at (0.00, 0.00)
- added H1: , ['lib_id', 'Connector_PinSocket_2.54mm:PinSocket_2x19_P2.54mm_Vertical'], F.Cu at (0.00, 0.00)
- added J1, J2, J6_1, J6_2, J6_3, J6_4: , ['lib_id', 'Connector_Phoenix:TerminalBlock_Phoenix_MKDS_1x2_P5.08mm_Horizontal'], F.Cu at (0.00, 0.00)
- added J3: , ['lib_id', 'Connector_PinHeader_2.54mm:PinHeader_1x05_P2.54mm_Vertical'], F.Cu at (0.00, 0.00)
- added J4: , ['lib_id', 'Connector_PinHeader_2.54mm:PinHeader_1x03_P2.54mm_Vertical'], F.Cu at (0.00, 0.00)
- added J5: , ['lib_id', 'Connector_PinHeader_2.54mm:PinHeader_1x04_P2.54mm_Vertical'], F.Cu at (0.00, 0.00)
- added Q1, Q2, Q3, Q4: , ['lib_id', 'TO-220-3_Vertical'], F.Cu at (0.00, 0.00)
- added R1, R2, R3, R4, R5, R6: , ['lib_id', 'R_Axial_DIN0207_L6.3mm_D2.5mm_P7.62mm_Horizontal'], F.Cu at (0.00, 0.00)
- added U1, U2: , ['lib_id', 'Connector_PinSocket_2.54mm:PinSocket_1x04_P2.54mm_Vertical'], F.Cu at (0.00, 0.00)
