File: kicad/ebike-bsd.kicad_sch (KiCad schematic)
At the start: 1 part

Commit message: kicad: 生成器改两路设计, 重新生成工程文件
generate_kicad.py:
- MOSFET 符号 Q1-Q4 → Q1-Q2 (V2.6 同侧前后并联)
- 删除 R3/R4 栅极电阻及 R3/R4 junction
- 原理图标签 LED_FL/FR/RL/RR → LED_LEFT/RIGHT
- 原理图连线删除 Q3/Q4 栅极和 J6_3/4 输出
- PCB net 列表精简 (28 → 21), tracks 删除 Q3/Q4 走线
- J5 连接器 4pin → 3pin (L/R/GND), J6 4 端子 → 2 端子
- 内嵌 BOM 模板同步两路

重新生成 kicad/ 下工程文件 (BOM/sch/pcb), 与脚本一致
Parts:
- ?: ['str', 'Reference'] ['str', 'J64'] -> ['str', 'J62']; ['str', 'Value'] ['str', 'TURN_RR'] -> ['str', 'TURN_RIGHT']
