File: kicad/ebike-bsd.kicad_sch (KiCad schematic)
At the start: 1 part

Commit message: Fix KiCad文件格式: 版本号20240108, 移除(str)包装, 兼容KiCad 8
Parts:
- removed ?: (no value)
- added D1: LED_LEFT, LED_THT:LED_D5.0mm, symbol Device:LED
- added D2: LED_RIGHT, LED_THT:LED_D5.0mm, symbol Device:LED
- added F1: F1, Fuse:Fuseholder_Cylinder-5x20mm_Wuerth_696103101002, symbol Device:Fuse
- added H1: ESP32-DevKitC, Connector_PinSocket_2.54mm:PinSocket_2x19_P2.54mm_Vertical, symbol Connector_Generic:Conn_02x19_Odd_Even
- added J1: 48V_INPUT, TerminalBlock:TerminalBlock_bornier-2_P5.08mm, symbol Connector_Generic:Conn_01x02
- added J2: 12V_OUT, TerminalBlock:TerminalBlock_bornier-2_P5.08mm, symbol Connector_Generic:Conn_01x02
- added J3: RADAR, Connector_PinHeader_2.54mm:PinHeader_1x05_P2.54mm_Vertical, symbol Connector_Generic:Conn_01x05
- added J4: BUZZER, Connector_PinHeader_2.54mm:PinHeader_1x03_P2.54mm_Vertical, symbol Connector_Generic:Conn_01x03
- added J5: SWITCH, Connector_PinHeader_2.54mm:PinHeader_1x04_P2.54mm_Vertical, symbol Connector_Generic:Conn_01x04
- added J61: TURN_FL, TerminalBlock:TerminalBlock_bornier-2_P5.08mm, symbol Connector_Generic:Conn_01x02
- added J62: TURN_FR, TerminalBlock:TerminalBlock_bornier-2_P5.08mm, symbol Connector_Generic:Conn_01x02
- added J63: TURN_RL, TerminalBlock:TerminalBlock_bornier-2_P5.08mm, symbol Connector_Generic:Conn_01x02
- added J64: TURN_RR, TerminalBlock:TerminalBlock_bornier-2_P5.08mm, symbol Connector_Generic:Conn_01x02
- added Q1: LED_FL, Package_TO_SOT_THT:TO-220-3_Vertical, symbol Transistor_FET:IRLZ44N
- added Q1, Q2, Q3, Q4: 100Ω, Resistor_THT:R_Axial_DIN0207_L6.3mm_D2.5mm_P7.62mm_Horizontal, symbol Device:R
- added Q2: LED_FR, Package_TO_SOT_THT:TO-220-3_Vertical, symbol Transistor_FET:IRLZ44N
- added Q3: LED_RL, Package_TO_SOT_THT:TO-220-3_Vertical, symbol Transistor_FET:IRLZ44N
- added Q4: LED_RR, Package_TO_SOT_THT:TO-220-3_Vertical, symbol Transistor_FET:IRLZ44N
- added R5, R6: 220Ω, Resistor_THT:R_Axial_DIN0207_L6.3mm_D2.5mm_P7.62mm_Horizontal, symbol Device:R
- added RPD1, RPD2, RPD3, RPD4: 10kΩ, Resistor_THT:R_Axial_DIN0207_L6.3mm_D2.5mm_P7.62mm_Horizontal, symbol Device:R
- added U1: XL7015, Module:XL7015, symbol Connector_Generic:Conn_01x04
- added U2: LM2596, Module:LM2596, symbol Connector_Generic:Conn_01x04
Other:
- company: (none) -> DIY
- title: (none) -> e-Bike BSD System
