File: kicad/ebike-bsd.kicad_sch (KiCad schematic)
At the start: 21 parts, among them J1 48V_INPUT, J2 12V_OUT, J3 RADAR, J4 BUZZER, J5 SWITCH, J6 C3_PANEL, J7 TURN_LAMPS, Q1 IRLZ44N, Q2 IRLZ44N, U1 XL7015_48-12V, U2 LM2596_12-5V

Commit message: fix: KiCad 10.0格式兼容 — 扁平坐标(at x y)+UUID+全局标签
Parts:
- F1: footprint Fuse:Fuseholder_Cylinder-5x20mm -> Fuseholder_Cylinder-5x20mm

Commit message: fix: 封装名兼容KiCad 10.0 — TerminalBlock_Phoenix + PinSocket
Parts:
- J1, J2: footprint TerminalBlock:TerminalBlock_bornier-2_P5.08mm -> TerminalBlock_Phoenix:TerminalBlock_Phoenix_MKDS_1x2_P5.08mm_Horizontal
- J7: footprint TerminalBlock:TerminalBlock_bornier-4_P5.08mm -> TerminalBlock_Phoenix:TerminalBlock_Phoenix_MKDS_1x4_P5.08mm_Horizontal
Changed lines of the file:
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@@
     (property "Reference" "J1" (id 0) (at 500 8150 0))
     (property "Value" "48V_INPUT" (id 1) (at 500 7850 0))
-    (property "Footprint" "TerminalBlock:TerminalBlock_bornier-2_P5.08mm" (id 2) (at 0 0 0) (hide yes))
+    (property "Footprint" "TerminalBlock_Phoenix:TerminalBlock_Phoenix_MKDS_1x2_P5.08mm_Horizontal" (id 2) (at 0 0 0) (hide yes))
     (pin "1")
     (pin "2")
@@
     (property "Reference" "J2" (id 0) (at 2600 7100 0))
     (property "Value" "12V_OUT" (id 1) (at 2600 6900 0))
-    (property "Footprint" "TerminalBlock:TerminalBlock_bornier-2_P5.08mm" (id 2) (at 0 0 0) (hide yes))
+    (property "Footprint" "TerminalBlock_Phoenix:TerminalBlock_Phoenix_MKDS_1x2_P5.08mm_Horizontal" (id 2) (at 0 0 0) (hide yes))
     (pin "1")
     (pin "2")
@@
     (property "Reference" "J7" (id 0) (at 7500 7150 0))
     (property "Value" "TURN_LAMPS" (id 1) (at 7500 6850 0))
-    (property "Footprint" "TerminalBlock:TerminalBlock_bornier-4_P5.08mm" (id 2) (at 0 0 0) (hide yes))
+    (property "Footprint" "TerminalBlock_Phoenix:TerminalBlock_Phoenix_MKDS_1x4_P5.08mm_Horizontal" (id 2) (at 0 0 0) (hide yes))
     (pin "1")
     (pin "2")
